File: power.kicad_sch (KiCad schematic)
At the start: 5 parts, among them J2 Conn_02x05_Odd_Even

Commit message: feat: add bq25887 connector
Parts:
- renumbered R9 to R10, R10 to R11, R11 to R9
Changed lines of the file:
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@@
 		(dnp no)
 		(fields_autoplaced yes)
-		(property "Reference" "R9"
+		(property "Reference" "R10"
 			(at 160.02 97.7899 0)
 			(effects
@@
 			(project "muty"
 				(path "/c2c8c614-99fc-45e9-8585-8c2a223a7e3c/f9a88ca2-69a8-42c3-a1ae-63cae6df6df1"
-					(reference "R9")
+					(reference "R10")
 					(unit 1)
 				)
@@
 		(dnp no)
 		(fields_autoplaced yes)
-		(property "Reference" "#PWR037"
+		(property "Reference" "#PWR038"
 			(at 176.53 97.79 0)
 			(effects
@@
 			(project "muty"
 				(path "/c2c8c614-99fc-45e9-8585-8c2a223a7e3c/f9a88ca2-69a8-42c3-a1ae-63cae6df6df1"
-					(reference "#PWR037")
+					(reference "#PWR038")
 					(unit 1)
 				)
@@
 		(dnp no)
 		(fields_autoplaced yes)
-		(property "Reference" "#PWR036"
+		(property "Reference" "#PWR037"
 			(at 170.18 55.88 0)
 			(effects
@@
 		)
 		(instances
-			(project ""
-				(path "/c2c8c614-99fc-45e9-8585-8c2a223a7e3c/f9a88ca2-69a8-42c3-a1ae-63cae6df6df1"
-					(reference "#PWR036")
+			(project "muty"
+				(path "/c2c8c614-99fc-45e9-8585-8c2a223a7e3c/f9a88ca2-69a8-42c3-a1ae-63cae6df6df1"
+					(reference "#PWR037")
 					(unit 1)
 				)
@@
 		)
 		(instances
-			(project ""
+			(project "muty"
 				(path "/c2c8c614-99fc-45e9-8585-8c2a223a7e3c/f9a88ca2-69a8-42c3-a1ae-63cae6df6df1"
 					(reference "J2")
@@
 		(dnp no)
 		(fields_autoplaced yes)
-		(property "Reference" "R11"
+		(property "Reference" "R9"
 			(at 149.86 116.8399 0)
 			(effects
@@
 			(project "muty"
 				(path "/c2c8c614-99fc-45e9-8585-8c2a223a7e3c/f9a88ca2-69a8-42c3-a1ae-63cae6df6df1"
-					(reference "R11")
+					(reference "R9")
 					(unit 1)
 				)
@@
 		)
 		(instances
-			(project ""
+			(project "muty"
 				(path "/c2c8c614-99fc-45e9-8585-8c2a223a7e3c/f9a88ca2-69a8-42c3-a1ae-63cae6df6df1"
 					(reference "R8")
@@
 		(on_board yes)
 		(dnp no)
-		(property "Reference" "#PWR038"
+		(property "Reference" "#PWR036"
 			(at 167.64 128.27 0)
 			(effects
@@
 			(project "muty"
 				(path "/c2c8c614-99fc-45e9-8585-8c2a223a7e3c/f9a88ca2-69a8-42c3-a1ae-63cae6df6df1"
-					(reference "#PWR038")
+					(reference "#PWR036")
 					(unit 1)
 				)
@@
 		(dnp no)
 		(fields_autoplaced yes)
-		(property "Reference" "R10"
+		(property "Reference" "R11"
 			(at 170.18 97.7899 0)
 			(effects
@@
 			(project "muty"
 				(path "/c2c8c614-99fc-45e9-8585-8c2a223a7e3c/f9a88ca2-69a8-42c3-a1ae-63cae6df6df1"
-					(reference "R10")
-					(unit 1)
-				)
+					(reference "R11")
+					(unit 1)
+				)
